File: CAN.sch (KiCad schematic (older format))
At the start: 23 parts, among them J4 CAN_Out, U4 ADM3055E, U5 CDSOT23-T24CAN

Commit message: Updates dashboard project to most recent version
Parts:
- removed J4: CAN_Out, UTSVT_Connectors:Molex_MicroFit3.0_1x4xP3.00mm_PolarizingPeg_Vertical, symbol utsvt-connectors:CANConnector
- removed R4: 60, Resistor_SMD:R_0805_2012Metric, symbol Device:R
- removed TP6: CAN_ISO_Vout, TestPoint:TestPoint_Keystone_5005-5009_Compact, symbol Connector:TestPoint
- removed TP7: CAN_ISO_Vin, TestPoint:TestPoint_Keystone_5005-5009_Compact, symbol Connector:TestPoint
- removed TP8: CAN_ISO_GndIn, TestPoint:TestPoint_Keystone_5005-5009_Compact, symbol Connector:TestPoint
- removed TP9: CAN_ISO_GndOut, TestPoint:TestPoint_Keystone_5005-5009_Compact, symbol Connector:TestPoint
- removed U4: ADM3055E, UTSVT_ICs:SOIC-20W_7.5x15.4mm_Pitch1.27mm, symbol utsvt-chips:ADM3055E
- removed U5: CDSOT23-T24CAN, Package_TO_SOT_SMD:SOT-23W, symbol utsvt-chips:CDSOT23-T24CAN
- added J19: CAN_IN, utsvt_conn:Molex_MicroFit3.0_1x4xP3.00mm_PolarizingPeg_Vertical, symbol Connector_Generic:Conn_01x04
- added J20: CAN_OUT, utsvt_conn:Molex_MicroFit3.0_1x4xP3.00mm_PolarizingPeg_Vertical, symbol Connector_Generic:Conn_01x04
- added U15: ADM3055E, utsvt_ics:SOIC-20W_7.5x15.4mm_Pitch1.27mm, symbol Chips:ADM3055E
- added U16: CDSOT23-T24CAN, Package_TO_SOT_SMD:SOT-23W, symbol Chips:CDSOT23-T24CAN
- C25: renamed from C18; Mouser Part Number (none) -> 80-C0805C106K8RAUTO
- C26: renamed from C19; Mouser Part Number (none) -> 80-C0805C104K3R
- C27: renamed from C20; Mouser Part Number (none) -> 80-C0805C104K3R
- C28: renamed from C21; Mouser Part Number (none) -> 80-C0805X103K1R3316
- C29: renamed from C22; value 10uF -> 0.22uF; Mouser Part Number (none) -> 80-C0805C224J1RECTU
- C30: renamed from C23; value 0.22uF -> 10uF; Mouser Part Number (none) -> 80-C0805C106K8RAUTO
- C31: renamed from C24; Mouser Part Number (none) -> 80-C0805C104K3R
- C32: renamed from C25; Mouser Part Number (none) -> 80-C0805X103K1R3316
- L5: renamed from L2; Mouser Part Number (none) -> 963-BK2125LM182-T
- L6: renamed from L3; Mouser Part Number (none) -> 963-BK2125LM182-T
- R32: renamed from R2; Mouser Part Number (none) -> 71-CRCW08050000Z0EAC
- R33: renamed from R3; value 60 -> 120; Mouser Part Number (none) -> 71-CRCW080559R0FKEA
- renumbered TP10 to TP7, TP11 to TP8
Connections:
- wire segments 104 -> 103
Other:
- note added: "As long as total equals to 120 Ohms,\nthe two termination resistors can be any value"
