File: CAN.sch (KiCad schematic (older format))
At the start: 18 parts, among them J19 CAN_IN, J20 CAN_OUT, J26 CAN_TP, U15 ADM3055E, U16 CDSOT23-T24CAN

Commit message: removes the isp
Parts:
- U15: symbol utsvt-chips:ADM3055E -> Dashboard-rescue:ADM3055E-utsvt-chips
- U16: symbol utsvt-chips:CDSOT23-T24CAN -> Dashboard-rescue:CDSOT23-T24CAN-utsvt-chips
Changed lines of the file:
@@
 $EndComp
 $Comp
-L utsvt-chips:ADM3055E U?
+L Dashboard-rescue:ADM3055E-utsvt-chips U?
 U 1 1 5F175F7A
 P 4350 3600
@@
 $EndComp
 $Comp
-L utsvt-chips:CDSOT23-T24CAN U?
+L Dashboard-rescue:CDSOT23-T24CAN-utsvt-chips U?
 U 1 1 5F177CC0
 P 8100 2850
