File: Dashboard.sch (KiCad schematic (older format))
At the start: 37 parts, among them J1 SWD, J10 Right Signal, J11 Brake Signal, J12 Headlight, J14 SPI3, J15 Vs-SPI1, J16 SPI1, J17 Vs-I2C3, J18 I2C3, J2 Logic Analyzer, J5 Array Contactor 1, J6 Motor Contactor 1, J7 Array Contactor 2, J8 Motor Contactor 2, J9 Left Signal, SW1 B3SL-1002P, U1 STM32F413RHTx, Y1 NX8045GB-8.000M-STD-CSJ-1

Commit message: Updates dashboard project to most recent version
Parts:
- removed C1, C3: 6pF, Capacitor_SMD:C_0805_2012Metric, symbol Device:C
- removed C10, C4: 0.1uF, Capacitor_SMD:C_0805_2012Metric, symbol Device:C
- removed C2: 2.2uF, Capacitor_SMD:C_0805_2012Metric, symbol Device:C
- removed J1: SWD, Connector_PinHeader_2.54mm:PinHeader_1x03_P2.54mm_Vertical, symbol Connector_Generic:Conn_01x03
- removed J10: Right Signal, UTSVT_Connectors:Molex_MicroFit3.0_1x2xP3.00mm_PolarizingPeg_Vertical, symbol Connector_Generic:Conn_01x02
- removed J11: Brake Signal, UTSVT_Connectors:Molex_MicroFit3.0_1x2xP3.00mm_PolarizingPeg_Vertical, symbol Connector_Generic:Conn_01x02
- removed J14: SPI3, Connector_Molex_Microfit:Molex_Micro-Fit_3.0_43650-0515_1x05_P3.00mm_Vertical, symbol Connector_Generic:Conn_01x05
- removed J15: Vs-SPI1, Connector_PinHeader_2.54mm:PinHeader_1x03_P2.54mm_Vertical, symbol Connector_Generic:Conn_01x03
- removed J16: SPI1, Connector_Molex_Microfit:Molex_Micro-Fit_3.0_43650-0515_1x05_P3.00mm_Vertical, symbol Connector_Generic:Conn_01x05
- removed J18: I2C3, UTSVT_Connectors:Molex_MicroFit3.0_1x4xP3.00mm_PolarizingPeg_Vertical, symbol Connector_Generic:Conn_01x04
- removed J2: Logic Analyzer, Connector_PinHeader_2.54mm:PinHeader_2x05_P2.54mm_Vertical, symbol Connector_Generic:Conn_02x05_Odd_Even
- removed J5: Array Contactor 1, UTSVT_Connectors:Molex_MicroFit3.0_1x4xP3.00mm_PolarizingPeg_Vertical, symbol Connector_Generic:Conn_01x04
- removed J6: Motor Contactor 1, UTSVT_Connectors:Molex_MicroFit3.0_1x4xP3.00mm_PolarizingPeg_Vertical, symbol Connector_Generic:Conn_01x04
- removed J7: Array Contactor 2, UTSVT_Connectors:Molex_MicroFit3.0_1x4xP3.00mm_PolarizingPeg_Vertical, symbol Connector_Generic:Conn_01x04
- removed J8: Motor Contactor 2, UTSVT_Connectors:Molex_MicroFit3.0_1x4xP3.00mm_PolarizingPeg_Vertical, symbol Connector_Generic:Conn_01x04
- removed J9: Left Signal, UTSVT_Connectors:Molex_MicroFit3.0_1x2xP3.00mm_PolarizingPeg_Vertical, symbol Connector_Generic:Conn_01x02
- removed MH1, MH2, MH3, MH4: MountingHole, MountingHole:MountingHole_3mm, symbol Mechanical:MountingHole
- removed R37, R38: 4.7k, Resistor_SMD:R_0805_2012Metric, symbol Device:R
- removed SW1: B3SL-1002P, Button_Switch_SMD:SW_SPST_B3SL-1002P, symbol Switch:SW_Push
- removed U1: STM32F413RHTx, Package_QFP:LQFP-64_10x10mm_P0.5mm, symbol MCU_ST_STM32F4:STM32F413RHTx
- added C1, C2, C3, C4: 1u, Capacitor_SMD:C_0805_2012Metric, symbol Device:C_Small
- added C10: 4.7uF, Capacitor_SMD:C_0805_2012Metric, symbol Device:C_Small
- added C14: 100nF, Capacitor_SMD:C_0805_2012Metric, symbol Device:C
- added C15: 1uF, Capacitor_SMD:C_0805_2012Metric, symbol Device:C
- added C16, C17, C18, C19: 0.1uF, Capacitor_SMD:C_0805_2012Metric, symbol Device:C
- added D1: LeftSignal, utsvt_conn:Molex_MicroFit3.0_1x2xP3.00mm_PolarizingPeg_Vertical, symbol Device:LED
- added D10, D11, D12, D13, D4, D5, D6, D7: D, Diode_SMD:D_0805_2012Metric, symbol Device:D
- added D2: RightSignal, utsvt_conn:Molex_MicroFit3.0_1x2xP3.00mm_PolarizingPeg_Vertical, symbol Device:LED
- added D3: KILL_SW_LED, utsvt_conn:Molex_MicroFit3.0_1x2xP3.00mm_PolarizingPeg_Vertical, symbol Device:LED
- added D8: MOTOR-PRECHARGE, utsvt_conn:Molex_MicroFit3.0_1x2xP3.00mm_PolarizingPeg_Vertical, symbol Device:LED
- added D9: ARRAY-PRECHARGE, utsvt_conn:Molex_MicroFit3.0_1x2xP3.00mm_PolarizingPeg_Vertical, symbol Device:LED
- added H1, H2, H3, H4, H5, H6, H7: MountingHole, MountingHole:MountingHole_3mm, symbol Mechanical:MountingHole
- added J1: Left_Signal, utsvt_conn:Molex_MicroFit3.0_1x2xP3.00mm_PolarizingPeg_Vertical, symbol Connector_Generic:Conn_01x02
- added J10, J11, J16: Conn_01x03_Female, utsvt_conn:Molex_MicroFit3.0_1x3xP3.00mm_PolarizingPeg_Vertical, symbol Connector_Generic:Conn_01x03
- added J13: Motor-P, utsvt_conn:Molex_MicroFit3.0_1x2xP3.00mm_PolarizingPeg_Vertical, symbol Connector_Generic:Conn_01x02
- added J14: Array-C, utsvt_conn:Molex_MicroFit3.0_1x2xP3.00mm_PolarizingPeg_Vertical, symbol Connector_Generic:Conn_01x02
- added J15: Array-P, utsvt_conn:Molex_MicroFit3.0_1x2xP3.00mm_PolarizingPeg_Vertical, symbol Connector_Generic:Conn_01x02
- added J2: Right_Signal, utsvt_conn:Molex_MicroFit3.0_1x2xP3.00mm_PolarizingPeg_Vertical, symbol Connector_Generic:Conn_01x02
- added J3: Brake Light, utsvt_conn:Molex_MicroFit3.0_1x2xP3.00mm_PolarizingPeg_Vertical, symbol Connector_Generic:Conn_01x02
- added J4: Headlight, utsvt_conn:Molex_MicroFit3.0_1x2xP3.00mm_PolarizingPeg_Vertical, symbol Connector_Generic:Conn_01x02
- added J5: LED_Cable, Connector_PinHeader_2.54mm:PinHeader_2x07_P2.54mm_Vertical, symbol Connector_Generic:Conn_01x11
- added J6: Backup, utsvt_conn:Molex_MicroFit3.0_1x2xP3.00mm_PolarizingPeg_Vertical, symbol Connector_Generic:Conn_01x02
- added J7: BPS_PWR, utsvt_conn:Molex_MicroFit3.0_1x2xP3.00mm_PolarizingPeg_Vertical, symbol Connector_Generic:Conn_01x02
- added J8: JTAG, Connector_PinHeader_2.54mm:PinHeader_1x06_P2.54mm_Vertical, symbol Connector_Generic:Conn_01x06
- added J9: Gecko_Cable, utsvt_conn:ribbon_cable_right_2x10, symbol Connector_Generic:Conn_02x10_Counter_Clockwise
- added L1, L2, L3, L4: 22u, Inductor_SMD:L_0805_2012Metric, symbol pspice:INDUCTOR
- added PS1, PS2, PS3, PS4: RCD-24, utsvt_special:RCD-24, symbol Dash:RCD-24
- added Q1, Q2, Q3, Q4: Q_PNP_BEC, Package_TO_SOT_SMD:SOT-23, symbol Device:Q_PNP_BEC
- added R1, R18, R19, R2, R20, R27, R28, R3, R6, R7: 10k, Resistor_SMD:R_0805_2012Metric, symbol Device:R_US
- added R10, R11, R8, R9: 105, Resistor_SMD:R_0805_2012Metric, symbol Device:R_US
- added R12: 1.2k, Resistor_SMD:R_0805_2012Metric, symbol Device:R_US
- added R13, R14, R21, R22: 330R, Resistor_SMD:R_0805_2012Metric, symbol Device:R_US
- added R15, R16, R17: 100k, Resistor_SMD:R_0805_2012Metric, symbol Device:R_Small_US
- added R23, R24, R25, R26: 105R, Resistor_SMD:R_0805_2012Metric, symbol Device:R_US
- added R4, R5: 4.9k, Resistor_SMD:R_0805_2012Metric, symbol Device:R_US
- added SW1: CRUISE_SET, utsvt_conn:Molex_MicroFit3.0_1x3xP3.00mm_PolarizingPeg_Vertical, symbol Switch:SW_SPDT
- added SW10: RESET, Button_Switch_SMD:SW_SPST_B3SL-1002P, symbol Switch:SW_SPST
- added SW2: CRUISE, utsvt_conn:Molex_MicroFit3.0_1x3xP3.00mm_PolarizingPeg_Vertical, symbol Switch:SW_SPDT
- added SW3: HAZARD, utsvt_conn:Molex_MicroFit3.0_1x3xP3.00mm_PolarizingPeg_Vertical, symbol Switch:SW_SPDT
- added SW4: HEADLIGHT_SW, utsvt_conn:Molex_MicroFit3.0_1x3xP3.00mm_PolarizingPeg_Vertical, symbol Switch:SW_SPDT
- added SW5: F/R_SW, utsvt_conn:Molex_MicroFit3.0_1x3xP3.00mm_PolarizingPeg_Vertical, symbol Switch:SW_SPDT
- added SW6: BACKUP_SW, utsvt_conn:Molex_MicroFit3.0_1x3xP3.00mm_PolarizingPeg_Vertical, symbol Switch:SW_SPDT
- added SW7: SW_Rotary2x6, utsvt_special:CK1035, symbol Switch:SW_Rotary2x6
- added SW8: TURN_SIGNAL_SW, utsvt_conn:Molex_MicroFit3.0_1x3xP3.00mm_PolarizingPeg_Vertical, symbol Switch:SW_SPDT_MSM
- added SW9: KILL_SW, utsvt_conn:Molex_MicroFit3.0_1x3xP3.00mm_PolarizingPeg_Vertical, symbol Switch:SW_SPDT
- added TP1: POWER, TestPoint:TestPoint_Keystone_5005-5009_Compact, symbol Connector:TestPoint
- added U1, U10, U11, U2, U3, U4, U5, U6, U8, U9: EL3H7, Package_SO:SOP-4_4.4x2.6mm_P1.27mm, symbol Isolator:SFH617A-1
- added U7: STM32F413RHTx, Package_QFP:LQFP-64_10x10mm_P0.5mm, symbol MCU_ST_STM32F4:STM32F413RHTx
- C11, C12, C5, C6: value 0.1uF -> 100nF; Mouser Part Number (none) -> 80-C0805C104K3R
- C13: Mouser Part Number (none) -> 80-C0805C475K3RAUTO
- C7, C8: value 0.1uF -> 12pF; Mouser Part Number (none) -> 80-C0805C479K1G
- C9: value 1uF -> 100nF; Mouser Part Number (none) -> 80-C0805C104K3R
- J12: value Headlight -> Motor-C; footprint UTSVT_Connectors:Molex_MicroFit3.0_1x2xP3.00mm_PolarizingPeg_Vertical -> utsvt_conn:Molex_MicroFit3.0_1x2xP3.00mm_PolarizingPeg_Vertical
- J17: value Vs-I2C3 -> Conn_01x03_Female; footprint Connector_PinHeader_2.54mm:PinHeader_1x03_P2.54mm_Vertical -> utsvt_conn:Molex_MicroFit3.0_1x3xP3.00mm_PolarizingPeg_Vertical
- Y1: value NX8045GB-8.000M-STD-CSJ-1 -> Crystal; footprint UTSVT_BPS:NX8045GB-8.000M-STD-CSJ-1 -> Crystal:Crystal_SMD_TXC_7A-2Pin_5x3.2mm
Connections:
- net labels added: +12V, A_CNCTR, A_PRCHG, Accel_Pot, Accel_Pot2, BK_LGHT, BPS_FAULT, BPS_PWR, Backup, Brake_Pot, Brake_Pot2, CRUZ_EN, CRUZ_ST, CTRL_FAULT, FR_SW, GNDA, GNDPWR, HZD_SW, HeadlightPWR, IG1, IG2, JTDI, JTDO, LEFT_BLINK, LEFT_SW, M_CNCTR, M_PRCHG, RIGHT_BLINK, RIGHT_SW, RSVD_LED, UART3_Tx
- net labels removed: AC1_CHECK, AC1_EN, AC2_CHECK, AC2_EN, Brake_Signal, CAN1_RX, CAN1_TX, Headlight, I2C3_SCL, I2C3_SDA, Left_Signal, MC1_CHECK, MC1_EN, MC2_CHECK, MC2_EN, OSC_IN, OSC_OUT, Right_Signal, SPI1_CLK, SPI1_MISO, SPI1_MOSI, SPI3_CLK, SPI3_MISO, SPI3_MOSI, UART1_RX, UART1_TX, array, bps, brake, chan1, chan2, cruise, decrease, hazard, increase, left, motor, regen, reverse, right, set-cancel, xtra1, xtra2, xtra3
- wire segments 230 -> 435
- no-connect marks 4 -> 38
Other:
- note added: "8M"
- note added: "All of these are negative logic LEDs\n"
- note added: "Are there better/cheaper\ndrivers?"
- note added: "Exterior Lights"
- note added: "For the boad itself"
- note added: "For the gecko\n"
- note added: "Ignition Switch"
- note added: "Potentiometers"
- note added: "Power state indicators"
- note added: "Should this be\nmale or female?"
- note added: "TODO: Assign pins for\n 1. BPS Fault\n 2. Control Fault\n 3. The Reserved Pin\nThe currently assigned pins should be considered temporary."
- note added: "TODO: Check to make sure\nthat all these switches have\nthe same "on" position."
- note added: "TODO: This connector was\noriginally the other way\naround. Will this still connect?"
- note added: "TODO: figure out which diodes\nthese are."
- note added: "TODO: make labels consistent.\nShould they be all UPPERCASE\nor Camel Case?"
- note added: "TODO: male or female?"
- note added: "TODO: should this be male or femal?"
- note added: "TODO: verify that this is all that needs to be done.\nRead the code to ensure all ports that are used are\non here.\n\nLook at all the other comments.\n\nAlso check over all the footprints again.\n\nAlso look at all the bodge wires running\naround the twins' board."
- note added: "These are negative-logic signals."
- note added: "Timing control for the lights"
- note added: "VDDA"
- note removed: "Bypass Capacitors"
- note removed: "Contactors"
- note removed: "Debug"
- note removed: "Header select\n"
- note removed: "I2C/SPI"
- note removed: "Isolated +5V and +3.3V.\nUse GND as common gnd for electronic components.\nConnect GNDPWR when using +12V."
- note removed: "Lights"
- note removed: "POWAH\n"
- note removed: "Place these capacitors as close to mcu as possible for correct operation.\nVDD/VSS"
- note removed: "Programming Pins."
- note removed: "SPI for screen. SPI for led. I2C incase"
- note removed: "Switches"
- note removed: "The crystal and caps have\nto be as close to the uC\nas possible."
- note removed: "VDDA/VSSA (VREF+/VREF-)"

Commit message: Edits schematic to make turn lights software controlled
Parts:
- removed D1: LeftSignal, utsvt_conn:Molex_MicroFit3.0_1x2xP3.00mm_PolarizingPeg_Vertical, symbol Device:LED
- removed D10, D11, D12, D13, D4, D5, D6, D7: D, Diode_SMD:D_0805_2012Metric, symbol Device:D
- removed D2: RightSignal, utsvt_conn:Molex_MicroFit3.0_1x2xP3.00mm_PolarizingPeg_Vertical, symbol Device:LED
- removed D8: MOTOR-PRECHARGE, utsvt_conn:Molex_MicroFit3.0_1x2xP3.00mm_PolarizingPeg_Vertical, symbol Device:LED
- removed D9: ARRAY-PRECHARGE, utsvt_conn:Molex_MicroFit3.0_1x2xP3.00mm_PolarizingPeg_Vertical, symbol Device:LED
- removed Q1, Q2, Q3, Q4: Q_PNP_BEC, Package_TO_SOT_SMD:SOT-23, symbol Device:Q_PNP_BEC
- removed R15, R16, R17: 100k, Resistor_SMD:R_0805_2012Metric, symbol Device:R_Small_US
- removed R21, R22: 330R, Resistor_SMD:R_0805_2012Metric, symbol Device:R_US
- added D1, D2, D4, D5: BAS70-04, Package_TO_SOT_SMD:SOT-23, symbol utsvt-chips:BAS70-04
- added J24: ExtraGPIO_Conn, Connector_PinHeader_2.54mm:PinHeader_1x07_P2.54mm_Vertical, symbol Connector_Generic:Conn_01x07
- added J25: UART_TP, Connector_PinHeader_2.54mm:PinHeader_1x02_P2.54mm_Vertical, symbol Connector_Generic:Conn_01x02
- added R15, R16: ?, Resistor_SMD:R_0805_2012Metric, symbol Device:R_US
- added TP11: RIGHT_BLINK, TestPoint:TestPoint_Pad_D1.5mm, symbol Connector:TestPoint
- added TP12: BK_LIGHT, TestPoint:TestPoint_Pad_D1.5mm, symbol Connector:TestPoint
- added TP7: Headlight_PWR, TestPoint:TestPoint_Pad_D1.5mm, symbol Connector:TestPoint
- added TP8: LEFT_BLINK, TestPoint:TestPoint_Pad_D1.5mm, symbol Connector:TestPoint
- D3, J1, J12, J13, J14, J15, J2, J3, J4, J6, J7: footprint utsvt_conn:Molex_MicroFit3.0_1x2xP3.00mm_PolarizingPeg_Vertical -> UTSVT_Connectors:Molex_MicroFit3.0_1x2xP3.00mm_PolarizingPeg_Vertical
- J10: value Conn_01x03_Female -> AccelConn; footprint utsvt_conn:Molex_MicroFit3.0_1x3xP3.00mm_PolarizingPeg_Vertical -> UTSVT_Connectors:Molex_MicroFit3.0_1x3xP3.00mm_PolarizingPeg_Vertical
- J11: value Conn_01x03_Female -> BrakeConn; footprint utsvt_conn:Molex_MicroFit3.0_1x3xP3.00mm_PolarizingPeg_Vertical -> UTSVT_Connectors:Molex_MicroFit3.0_1x3xP3.00mm_PolarizingPeg_Vertical
- J16: value Conn_01x03_Female -> AccelConn2; footprint utsvt_conn:Molex_MicroFit3.0_1x3xP3.00mm_PolarizingPeg_Vertical -> UTSVT_Connectors:Molex_MicroFit3.0_1x3xP3.00mm_PolarizingPeg_Vertical
- J17: value Conn_01x03_Female -> BrakeConn2; footprint utsvt_conn:Molex_MicroFit3.0_1x3xP3.00mm_PolarizingPeg_Vertical -> UTSVT_Connectors:Molex_MicroFit3.0_1x3xP3.00mm_PolarizingPeg_Vertical
- R13, R14: value 330R -> ?; Mouser Part Number 71-CRCW0805330RFKEAC -> 71-CRCW080510K0FKEAC
- SW1, SW2, SW3, SW4, SW5, SW6, SW8, SW9: footprint utsvt_conn:Molex_MicroFit3.0_1x3xP3.00mm_PolarizingPeg_Vertical -> UTSVT_Connectors:Molex_MicroFit3.0_1x3xP3.00mm_PolarizingPeg_Vertical
- TP1: footprint TestPoint:TestPoint_Keystone_5005-5009_Compact -> TestPoint:TestPoint_Pad_1.5x1.5mm
Connections:
- net +3V3: now also D1.2, D2.2, D4.2, D5.2, R15.1; no longer R14.1
- net Accel_Pot: now also R14.1, D1.3, D1.3
- net Accel_Pot2: now also D4.3, D4.3, R16.1
- net BK_LGHT: now also U7.20 (PA4), TP12.1; no longer U7.14 (PA0)
- net Brake_Pot: now also R13.2, D2.3, D2.3
- net Brake_Pot2: now also D5.3, D5.3, R15.2
- net GND: now also R14.2, D1.1, D2.1, D4.1, D5.1, R16.2
- net HZD_SW: now also U7.62 (PB9)
- net HeadlightPWR: now also TP7.1
- net LEFT_BLINK: now also U7.14 (PA0), TP8.1
- net RIGHT_BLINK: now also U7.15 (PA1), TP11.1
- net UART3_Tx: now also J25.1 (Pin_1)
- net PC6: now reaches U7.37 (PC6)
- net PC6: now also J24.1 (Pin_1)
- net PC7: now reaches U7.38 (PC7)
- net PC7: now also J24.2 (Pin_2)
- net PC8: now reaches U7.39 (PC8)
- net PC8: now also J24.3 (Pin_3)
- net PC9: now reaches U7.40 (PC9)
- net PC9: now also J24.4 (Pin_4)
- net PA8: now reaches U7.41 (PA8)
- net PA8: now also J24.5 (Pin_5)
- net PA9: now reaches U7.42 (PA9)
- net PA9: now also J24.6 (Pin_6)
- net PA10: now reaches U7.43 (PA10)
- net PA10: now also J24.7 (Pin_7)
- net Motor-CAN/CAN_RX renamed Motor_CAN/CAN_RX
- net Motor-CAN/CAN_TX renamed Motor_CAN/CAN_TX
- net sheet5F7A9234/UART_RX renamed UART3_Rx
- net UART3_Rx: now also J25.2 (Pin_2)
- no-connect marks 38 -> 28
Other:
- note added: "Add test points\n"
- note added: "Change one CAN connector to the 5 pin connector \nhttps://www.digikey.com/product-detail/en/te-connectivity-amp-connectors/4-2172079-2/A120861-ND/5118755"
- note removed: "Timing control for the lights"

Commit message: Updates PCB to add changes from the schematic
Parts:
- J9: footprint utsvt_conn:ribbon_cable_right_2x10 -> UTSVT_Connectors:ribbon_cable_right_2x10
- PS1, PS2, PS3, PS4: footprint utsvt_special:RCD-24 -> UTSVT_Special:RCD-24
- SW7: footprint utsvt_special:CK1035 -> UTSVT_Special:CK1035
Changed lines of the file:
@@
 F 0 "SW7" H 3750 8875 50  0000 C CNN
 F 1 "SW_Rotary2x6" H 3750 8966 50  0000 C CNN
-F 2 "utsvt_special:CK1035" H 3600 10300 50  0001 C CNN
+F 2 "UTSVT_Special:CK1035" H 3600 10300 50  0001 C CNN
 F 3 "https://www.mouser.com/datasheet/2/242/CK-681.pdf" H 3600 10300 50  0001 C CNN
 F 4 "10WA325 " H 3700 9700 50  0001 C CNN "Mouser Part Number"
@@
 F 0 "J9" H 14500 6200 50  0000 C CNN
 F 1 "Gecko_Cable" H 14450 6100 50  0000 C CNN
-F 2 "utsvt_conn:ribbon_cable_right_2x10" H 15100 6050 50  0001 C CNN
+F 2 "UTSVT_Connectors:ribbon_cable_right_2x10" H 15100 6050 50  0001 C CNN
 F 3 "~" H 15100 6050 50  0001 C CNN
 F 4 "517-N2520-5002RB " H 15100 6050 50  0001 C CNN "Mouser Part Number"
@@
 F 0 "PS1" H 1750 1765 50  0000 C CNN
 F 1 "RCD-24" H 1750 1674 50  0000 C CNN
-F 2 "utsvt_special:RCD-24" H 1750 1350 50  0001 C CNN
+F 2 "UTSVT_Special:RCD-24" H 1750 1350 50  0001 C CNN
 F 3 "" H 1750 1350 50  0001 C CNN
 	1    1750 1350
@@
 F 0 "PS2" H 1750 2715 50  0000 C CNN
 F 1 "RCD-24" H 1750 2624 50  0000 C CNN
-F 2 "utsvt_special:RCD-24" H 1750 2300 50  0001 C CNN
+F 2 "UTSVT_Special:RCD-24" H 1750 2300 50  0001 C CNN
 F 3 "" H 1750 2300 50  0001 C CNN
 	1    1750 2300
@@
 F 0 "PS3" H 1750 3665 50  0000 C CNN
 F 1 "RCD-24" H 1750 3574 50  0000 C CNN
-F 2 "utsvt_special:RCD-24" H 1750 3250 50  0001 C CNN
+F 2 "UTSVT_Special:RCD-24" H 1750 3250 50  0001 C CNN
 F 3 "" H 1750 3250 50  0001 C CNN
 	1    1750 3250
@@
 F 0 "PS4" H 1750 4615 50  0000 C CNN
 F 1 "RCD-24" H 1750 4524 50  0000 C CNN
-F 2 "utsvt_special:RCD-24" H 1750 4200 50  0001 C CNN
+F 2 "UTSVT_Special:RCD-24" H 1750 4200 50  0001 C CNN
 F 3 "" H 1750 4200 50  0001 C CNN
 	1    1750 4200

Commit message: Organizes the schematic into hierarchical sheets
Parts:
- removed C1, C2, C3, C4: 1u, Capacitor_SMD:C_0805_2012Metric, symbol Device:C_Small
- removed C16, C17, C18, C19: 0.1uF, Capacitor_SMD:C_0805_2012Metric, symbol Device:C
- removed D1, D2, D4, D5: BAS70-04, Package_TO_SOT_SMD:SOT-23, symbol utsvt-chips:BAS70-04
- removed D3: KILL_SW_LED, UTSVT_Connectors:Molex_MicroFit3.0_1x2xP3.00mm_PolarizingPeg_Vertical, symbol Device:LED
- removed J1: Left_Signal, UTSVT_Connectors:Molex_MicroFit3.0_1x2xP3.00mm_PolarizingPeg_Vertical, symbol Connector_Generic:Conn_01x02
- removed J10: AccelConn, UTSVT_Connectors:Molex_MicroFit3.0_1x3xP3.00mm_PolarizingPeg_Vertical, symbol Connector_Generic:Conn_01x03
- removed J11: BrakeConn, UTSVT_Connectors:Molex_MicroFit3.0_1x3xP3.00mm_PolarizingPeg_Vertical, symbol Connector_Generic:Conn_01x03
- removed J12: Motor-C, UTSVT_Connectors:Molex_MicroFit3.0_1x2xP3.00mm_PolarizingPeg_Vertical, symbol Connector_Generic:Conn_01x02
- removed J13: Motor-P, UTSVT_Connectors:Molex_MicroFit3.0_1x2xP3.00mm_PolarizingPeg_Vertical, symbol Connector_Generic:Conn_01x02
- removed J14: Array-C, UTSVT_Connectors:Molex_MicroFit3.0_1x2xP3.00mm_PolarizingPeg_Vertical, symbol Connector_Generic:Conn_01x02
- removed J15: Array-P, UTSVT_Connectors:Molex_MicroFit3.0_1x2xP3.00mm_PolarizingPeg_Vertical, symbol Connector_Generic:Conn_01x02
- removed J16: AccelConn2, UTSVT_Connectors:Molex_MicroFit3.0_1x3xP3.00mm_PolarizingPeg_Vertical, symbol Connector_Generic:Conn_01x03
- removed J17: BrakeConn2, UTSVT_Connectors:Molex_MicroFit3.0_1x3xP3.00mm_PolarizingPeg_Vertical, symbol Connector_Generic:Conn_01x03
- removed J2: Right_Signal, UTSVT_Connectors:Molex_MicroFit3.0_1x2xP3.00mm_PolarizingPeg_Vertical, symbol Connector_Generic:Conn_01x02
- removed J3: Brake Light, UTSVT_Connectors:Molex_MicroFit3.0_1x2xP3.00mm_PolarizingPeg_Vertical, symbol Connector_Generic:Conn_01x02
- removed J4: Headlight, UTSVT_Connectors:Molex_MicroFit3.0_1x2xP3.00mm_PolarizingPeg_Vertical, symbol Connector_Generic:Conn_01x02
- removed J6: Backup, UTSVT_Connectors:Molex_MicroFit3.0_1x2xP3.00mm_PolarizingPeg_Vertical, symbol Connector_Generic:Conn_01x02
- removed J7: BPS_PWR, UTSVT_Connectors:Molex_MicroFit3.0_1x2xP3.00mm_PolarizingPeg_Vertical, symbol Connector_Generic:Conn_01x02
- removed L1, L2, L3, L4: 22u, Inductor_SMD:L_0805_2012Metric, symbol pspice:INDUCTOR
- removed PS1, PS2, PS3, PS4: RCD-24, UTSVT_Special:RCD-24, symbol Dash:RCD-24
- removed R1, R19, R2, R20, R27, R28, R3, R6, R7: 10k, Resistor_SMD:R_0805_2012Metric, symbol Device:R_US
- removed R10, R11, R8, R9: 105, Resistor_SMD:R_0805_2012Metric, symbol Device:R_US
- removed R12: 1.2k, Resistor_SMD:R_0805_2012Metric, symbol Device:R_US
- removed R13, R14, R15, R16: ?, Resistor_SMD:R_0805_2012Metric, symbol Device:R_US
- removed R23, R24, R25, R26: 105R, Resistor_SMD:R_0805_2012Metric, symbol Device:R_US
- removed R4, R5: 4.9k, Resistor_SMD:R_0805_2012Metric, symbol Device:R_US
- removed SW1: CRUISE_SET, UTSVT_Connectors:Molex_MicroFit3.0_1x3xP3.00mm_PolarizingPeg_Vertical, symbol Switch:SW_SPDT
- removed SW2: CRUISE, UTSVT_Connectors:Molex_MicroFit3.0_1x3xP3.00mm_PolarizingPeg_Vertical, symbol Switch:SW_SPDT
- removed SW3: HAZARD, UTSVT_Connectors:Molex_MicroFit3.0_1x3xP3.00mm_PolarizingPeg_Vertical, symbol Switch:SW_SPDT
- removed SW4: HEADLIGHT_SW, UTSVT_Connectors:Molex_MicroFit3.0_1x3xP3.00mm_PolarizingPeg_Vertical, symbol Switch:SW_SPDT
- removed SW5: F/R_SW, UTSVT_Connectors:Molex_MicroFit3.0_1x3xP3.00mm_PolarizingPeg_Vertical, symbol Switch:SW_SPDT
- removed SW6: BACKUP_SW, UTSVT_Connectors:Molex_MicroFit3.0_1x3xP3.00mm_PolarizingPeg_Vertical, symbol Switch:SW_SPDT
- removed SW7: SW_Rotary2x6, UTSVT_Special:CK1035, symbol Switch:SW_Rotary2x6
- removed SW8: TURN_SIGNAL_SW, UTSVT_Connectors:Molex_MicroFit3.0_1x3xP3.00mm_PolarizingPeg_Vertical, symbol Switch:SW_SPDT_MSM
- removed SW9: KILL_SW, UTSVT_Connectors:Molex_MicroFit3.0_1x3xP3.00mm_PolarizingPeg_Vertical, symbol Switch:SW_SPDT
- removed TP1: POWER, TestPoint:TestPoint_Pad_1.5x1.5mm, symbol Connector:TestPoint
- removed TP11: RIGHT_BLINK, TestPoint:TestPoint_Pad_D1.5mm, symbol Connector:TestPoint
- removed TP12: BK_LIGHT, TestPoint:TestPoint_Pad_D1.5mm, symbol Connector:TestPoint
- removed TP7: Headlight_PWR, TestPoint:TestPoint_Pad_D1.5mm, symbol Connector:TestPoint
- removed TP8: LEFT_BLINK, TestPoint:TestPoint_Pad_D1.5mm, symbol Connector:TestPoint
- removed U1, U10, U11, U2, U3, U4, U5, U6, U8, U9: EL3H7, Package_SO:SOP-4_4.4x2.6mm_P1.27mm, symbol Isolator:SFH617A-1
- added LOGO1: Dr. Hallock, UTSVT_Special:Hallock_Image_Small, symbol utsvt-misc:Logo_Placeholder
- added LOGO2: UTSVT, UTSVT_Special:UTSVT_Logo_Symbol, symbol utsvt-misc:Logo_Placeholder
Connections:
- net PA2: now reaches J9.17 (Pin_17), U7.16 (PA2)
- net PA3: now reaches J9.16 (Pin_16), U7.17 (PA3)
- net Headlight_SW: now reaches U7.24 (PC4)
- net BK_LGHT renamed BK_LIGHT
- net Car-CAN/CAN_RX renamed CAN_Rx
- net Car-CAN/CAN_TX renamed CAN_Tx
- net HeadlightPWR renamed Headlight_ON
- net Motor_CAN/CAN_RX renamed MotorCAN_Rx
- net Motor_CAN/CAN_TX renamed MotorCAN_Tx
- no-connect marks 28 -> 21
Other:
- note added: "Logo Placeholders"
- note removed: "Add test points\n"
- note removed: "Are there better/cheaper\ndrivers?"
- note removed: "Change one CAN connector to the 5 pin connector \nhttps://www.digikey.com/product-detail/en/te-connectivity-amp-connectors/4-2172079-2/A120861-ND/5118755"
- note removed: "Exterior Lights"
- note removed: "Ignition Switch"
- note removed: "Potentiometers"
- note removed: "Power state indicators"
- note removed: "Should this be\nmale or female?"
- note removed: "TODO: Check to make sure\nthat all these switches have\nthe same "on" position."
- note removed: "TODO: This connector was\noriginally the other way\naround. Will this still connect?"
- note removed: "TODO: figure out which diodes\nthese are."
- note removed: "TODO: male or female?"
- note removed: "TODO: should this be male or femal?"
- note removed: "These are negative-logic signals."
- moved on the sheet: C10, C11, C12, C13, C14, C15, C5, C6, C7, C8, C9, H1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
