File: USB.sch (KiCad schematic (older format))
At the start: 8 parts, among them J23 USB_B_Micro, U19 CP2102N-A01-GQFN24

Commit message: USB Tx/Rx, Crystal Keepout, 12V Separation, Can2-Can3, Motor CAN bus labels, Power Input Protection Circuitry
Parts:
- J23: symbol Connector:USB_B_Micro -> Dashboard-rescue:USB_B_Micro-Connector
Changed lines of the file:
@@
 $Descr A4 11693 8268
 encoding utf-8
-Sheet 4 10
+Sheet 10 10
 Title ""
 Date ""
@@
 $EndComp
 $Comp
-L Connector:USB_B_Micro J?
+L Dashboard-rescue:USB_B_Micro-Connector J?
 U 1 1 5C4964BB
 P 3000 4300
 AR Path="/5E91171A/5C4964BB" Ref="J?"  Part="1"
 AR Path="/5F7A9238/5C4964BB" Ref="J23"  Part="1"
+AR Path="/5C4964BB" Ref="J23"  Part="1"
 F 0 "J23" H 3000 4750 50  0000 C CNN
 F 1 "USB_B_Micro" H 3000 4650 50  0000 C CNN
