File: Potentiometers.kicad_sch (KiCad schematic)
At the start: 14 parts, among them J12 Brake_Sw, J7 Accel_Pot, J9 Brake_Pot

Commit message: Updated comments.
Other:
- note added: "Added brake pot, updated accel pot resistor values"
- note removed: "No change required"
Changed lines of the file:
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@@
 		)
 	)
-	(text "No change required\n"
+	(text "Added brake pot, updated accel pot resistor values"
 		(exclude_from_sim no)
-		(at 13.97 22.86 0)
+		(at 177.8 180.086 0)
 		(effects
 			(font
 				(face "KiCad Font")
-				(size 5 5)
-				(thickness 1)
-				(bold yes)
+				(size 1.524 1.524)
+				(thickness 0.1905)
 				(color 255 2 13 1)
 			)
