File: Potentiometers.kicad_sch (KiCad schematic)
At the start: 15 parts, among them J12 Brake_Sw, J7 Accel_Pot, J9 Brake Pos. Sensor

Commit message: Added part numbers wheeeeeeeeeeeeeeeeeeeee
Parts:
- C1: JLCPCB# (none) -> C28323
- C16: JLCPCB# (none) -> C28233
- C3: JLCPCB# (none) -> C1791; P/N pickle -> C0805C102K5GECAUTO
- D2: JLCPCB# (none) -> C2959841
- D3, D5: JLCPCB# (none) -> C23848
- R13: JLCPCB# (none) -> C17477
- R14: JLCPCB# (none) -> C149504
- R15: JLCPCB# (none) -> C17763; P/N CRCW08054K99FKEAC -> CRCW080559K0FKEA
- R16: JLCPCB# (none) -> C17477; P/N pickle -> RC0805JR-070RL
- R26, R27: JLCPCB# (none) -> C17414
Changed lines of the file:
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@@
+			)
+		)
+		(property "JLCPCB#" "C2959841"
+			(at 80.01 100.33 0)
+			(effects
+				(font
+					(size 1.27 1.27)
+				)
+				(hide yes)
 			)
 		)
@@
 			)
 		)
+		(property "JLCPCB#" "C28233"
+			(at 62.23 100.33 0)
+			(effects
+				(font
+					(size 1.27 1.27)
+				)
+				(hide yes)
+			)
+		)
 		(pin "1"
 		)
@@
 			)
 		)
+		(property "JLCPCB#" "C2959841"
+			(at 80.01 91.44 0)
+			(effects
+				(font
+					(size 1.27 1.27)
+				)
+				(hide yes)
+			)
+		)
 		(pin "2"
 		)
@@
 			)
 		)
-		(property "P/N" "CRCW08054K99FKEAC "
+		(property "P/N" "CRCW080559K0FKEA"
+			(at 88.9 96.52 0)
+			(effects
+				(font
+					(size 1.27 1.27)
+				)
+				(hide yes)
+			)
+		)
+		(property "JLCPCB#" "C17763"
 			(at 88.9 96.52 0)
 			(effects
@@
 		)
 		(property "P/N" "CRCW0805100KFKEAC"
+			(at 72.39 100.33 0)
+			(effects
+				(font
+					(size 1.27 1.27)
+				)
+				(hide yes)
+			)
+		)
+		(property "JLCPCB#" "C149504"
 			(at 72.39 100.33 0)
 			(effects
@@
 			)
 		)
+		(property "JLCPCB#" "C23848"
+			(at 226.06 115.57 0)
+			(effects
+				(font
+					(size 1.27 1.27)
+				)
+				(hide yes)
+			)
+		)
 		(pin "1"
 		)
@@
 			)
 		)
+		(property "JLCPCB#" "C17477"
+			(at 198.12 111.76 0)
+			(effects
+				(font
+					(size 1.27 1.27)
+				)
+				(hide yes)
+			)
+		)
 		(pin "2"
 		)
@@
 			)
 		)
+		(property "JLCPCB#" "C23848"
+			(at 226.06 107.95 0)
+			(effects
+				(font
+					(size 1.27 1.27)
+				)
+				(hide yes)
+			)
+		)
 		(pin "1"
 		)
@@
 			)
 		)
-		(property "P/N" "pickle"
+		(property "P/N" " RC0805JR-070RL"
+			(at 203.2 116.84 0)
+			(effects
+				(font
+					(size 1.27 1.27)
+				)
+				(hide yes)
+			)
+		)
+		(property "JLCPCB#" "C17477"
 			(at 203.2 116.84 0)
 			(effects
@@
 			)
 		)
+		(property "JLCPCB#" "C28323"
+			(at 78.74 148.59 0)
+			(effects
+				(font
+					(size 1.27 1.27)
+				)
+				(hide yes)
+			)
+		)
 		(pin "1"
 		)
@@
 			)
 		)
+		(property "JLCPCB#" "C17414"
+			(at 92.71 148.59 0)
+			(effects
+				(font
+					(size 1.27 1.27)
+				)
+				(hide yes)
+			)
+		)
 		(pin "1"
 		)
@@
 			)
 		)
-		(property "P/N" "pickle"
+		(property "P/N" "C0805C102K5GECAUTO"
+			(at 217.17 115.57 0)
+			(effects
+				(font
+					(size 1.27 1.27)
+				)
+				(hide yes)
+			)
+		)
+		(property "JLCPCB#" "C1791"
 			(at 217.17 115.57 0)
 			(effects
@@
 			)
 		)
+		(property "JLCPCB#" ""
+			(at 107.95 139.7 0)
+			(effects
+				(font
+					(size 1.27 1.27)
+				)
+				(hide yes)
+			)
+		)
 		(pin "1"
 		)
@@
 		)
 		(property "P/N" "430450626"
+			(at 176.53 111.76 0)
+			(effects
+				(font
+					(size 1.27 1.27)
+				)
+				(hide yes)
+			)
+		)
+		(property "JLCPCB#" ""
 			(at 176.53 111.76 0)
 			(effects
@@
 			)
 		)
+		(property "JLCPCB#" "C17414"
+			(at 85.09 142.24 0)
+			(effects
+				(font
+					(size 1.27 1.27)
+				)
+				(hide yes)
+			)
+		)
 		(pin "1"
 		)
@@
 			(at 123.19 96.52 0)
 			(effects
+				(font
+					(size 1.27 1.27)
+				)
+				(hide yes)
+			)
+		)
+		(property "JLCPCB#" ""
+			(at 123.19 96.52 0)
+			(effects
