File: Contactors.kicad_sch (KiCad schematic)
At the start: 9 parts, among them J10 A_PRCHG_BYPASS, J11 M_PRCHG_BYPASS, J17 M_CNTCTR, U10 EL3H7, U8 EL3H7, U9 EL3H7

Commit message: Updated comments.
Other:
- note added: "Added Motor_Contactor"
- note removed: "No change required"
Changed lines of the file:
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@@
 		)
 	)
-	(text "No change required\n"
+	(text "Added Motor_Contactor"
 		(exclude_from_sim no)
-		(at 15.24 22.86 0)
+		(at 178.054 180.086 0)
 		(effects
 			(font
 				(face "KiCad Font")
-				(size 5 5)
-				(thickness 1)
-				(bold yes)
+				(size 1.524 1.524)
+				(thickness 0.1905)
 				(color 255 2 13 1)
 			)

Commit message: Filled in part numbers, exported BOM and made Excel file for working with it.
Parts:
- J10, J11, J17: P/N 43650-0215 -> 436500244
- R24, R25, R32: P/N (none) -> CRCW0805105RFKEA
- U10, U8, U9: P/N (none) -> EL3H7DTAVG
Changed lines of the file:
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@@
+			)
+		)
+		(property "P/N" "EL3H7DTAVG "
+			(at 138.43 140.97 0)
+			(effects
+				(font
+					(size 1.27 1.27)
+				)
+				(hide yes)
 			)
 		)
@@
 			)
 		)
+		(property "P/N" "CRCW0805105RFKEA "
+			(at 124.46 138.43 0)
+			(effects
+				(font
+					(size 1.27 1.27)
+				)
+				(hide yes)
+			)
+		)
 		(pin "1"
 		)
@@
 			)
 		)
+		(property "P/N" "EL3H7DTAVG "
+			(at 138.43 64.77 0)
+			(effects
+				(font
+					(size 1.27 1.27)
+				)
+				(hide yes)
+			)
+		)
 		(pin "1"
 		)
@@
 			)
 		)
+		(property "P/N" "CRCW0805105RFKEA "
+			(at 124.46 62.23 0)
+			(effects
+				(font
+					(size 1.27 1.27)
+				)
+				(hide yes)
+			)
+		)
 		(pin "1"
 		)
@@
 		)
 		(property "Vds" ""
+			(at 124.46 101.6 0)
+			(effects
+				(font
+					(size 1.27 1.27)
+				)
+				(hide yes)
+			)
+		)
+		(property "P/N" "CRCW0805105RFKEA "
 			(at 124.46 101.6 0)
 			(effects
@@
 			)
 		)
-		(property "P/N" "43650-0215"
+		(property "P/N" "436500244"
 			(at 158.75 106.68 0)
 			(effects
@@
 		)
 		(property "Vds" ""
+			(at 138.43 104.14 0)
+			(effects
+				(font
+					(size 1.27 1.27)
+				)
+				(hide yes)
+			)
+		)
+		(property "P/N" "EL3H7DTAVG "
 			(at 138.43 104.14 0)
 			(effects
@@
 			)
 		)
-		(property "P/N" "43650-0215"
+		(property "P/N" "436500244"
 			(at 158.75 67.31 0)
 			(effects
@@
 			)
 		)
-		(property "P/N" "43650-0215"
+		(property "P/N" "436500244"
 			(at 160.02 143.51 0)
 			(effects
