File: Lights_Drivers.kicad_sch (KiCad schematic)
At the start: 15 parts, among them Q1 IRLML0030, Q3 IRLML0030, Q4 IRLML0030, U25 EL3H7, U26 EL3H7, U3 EL3H7

Commit message: Filled in part numbers, exported BOM and made Excel file for working with it.
Parts:
- R11, R12, R6: P/N (none) -> CRCW0805510RFKEAC
- R41, R56, R58: P/N (none) -> CRCW0805100KFKEAC
- U25, U26, U3: P/N (none) -> EL3H7DTAVG
Changed lines of the file:
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@@
+			)
+		)
+		(property "P/N" "EL3H7DTAVG "
+			(at 208.28 104.14 0)
+			(effects
+				(font
+					(size 1.27 1.27)
+				)
+				(hide yes)
 			)
 		)
@@
 			)
 		)
+		(property "P/N" "CRCW0805510RFKEAC"
+			(at 191.77 58.42 0)
+			(effects
+				(font
+					(size 1.27 1.27)
+				)
+				(hide yes)
+			)
+		)
 		(pin "1"
 		)
@@
 			)
 		)
+		(property "P/N" "EL3H7DTAVG "
+			(at 72.39 107.95 0)
+			(effects
+				(font
+					(size 1.27 1.27)
+				)
+				(hide yes)
+			)
+		)
 		(pin "1"
 		)
@@
 			)
 		)
+		(property "P/N" "CRCW0805510RFKEAC"
+			(at 193.04 101.6 0)
+			(effects
+				(font
+					(size 1.27 1.27)
+				)
+				(hide yes)
+			)
+		)
 		(pin "1"
 		)
@@
 			)
 		)
+		(property "P/N" "CRCW0805100KFKEAC"
+			(at 82.55 116.84 0)
+			(effects
+				(font
+					(size 1.27 1.27)
+				)
+				(hide yes)
+			)
+		)
 		(pin "2"
 		)
@@
 		)
 		(property "Vds" ""
+			(at 207.01 60.96 0)
+			(effects
+				(font
+					(size 1.27 1.27)
+				)
+				(hide yes)
+			)
+		)
+		(property "P/N" "EL3H7DTAVG "
 			(at 207.01 60.96 0)
 			(effects
@@
 			)
 		)
+		(property "P/N" "CRCW0805100KFKEAC"
+			(at 218.44 113.03 0)
+			(effects
+				(font
+					(size 1.27 1.27)
+				)
+				(hide yes)
+			)
+		)
 		(pin "2"
 		)
@@
 			)
 		)
-		(property "Datasheet" "~"
+		(property "Datasheet" "https://www.molex.com/en-us/products/part-detail/436500215"
 			(at 234.95 101.6 0)
 			(effects
@@
 			)
 		)
-		(property "Datasheet" "~"
+		(property "Datasheet" "https://www.molex.com/en-us/products/part-detail/436500215"
 			(at 233.68 58.42 0)
 			(effects
@@
 			)
 		)
+		(property "P/N" "CRCW0805510RFKEAC"
+			(at 53.34 105.41 0)
+			(effects
+				(font
+					(size 1.27 1.27)
+				)
+				(hide yes)
+			)
+		)
 		(pin "2"
 		)
@@
 			)
 		)
+		(property "P/N" "CRCW0805100KFKEAC"
+			(at 217.17 69.85 0)
+			(effects
+				(font
+					(size 1.27 1.27)
+				)
+				(hide yes)
+			)
+		)
 		(pin "2"
 		)
@@
 			)
 		)
-		(property "Datasheet" "~"
+		(property "Datasheet" "https://www.molex.com/en-us/products/part-detail/436500215"
 			(at 99.06 105.41 0)
 			(effects
