File: Controls-Leader.kicad_sch (KiCad schematic)
At the start: 49 parts, among them J1 ExtraADCs, J10 Dashboard_TPs, J13 UART_TP, J15 Pot_TPs, J2 UART_TP, J25 UART_TP, J3 ExtraGPIO_Conn, J8 SWD, SW10 RESET, U7 STM32F413RHTx, Y1 Crystal

Commit message: I think the silkscreen is okay now.
Parts:
- J1: footprint UTSVT_Connectors:Molex_MicroFit3.0_1x3xP3.00mm_PolarizingPeg_Vertical -> Connector_PinHeader_2.54mm:PinHeader_1x03_P2.54mm_Vertical
- J10: footprint UTSVT_Connectors:Molex_MicroFit3.0_2x6xP3.00mm_PolarizingPeg_Vertical -> Connector_PinHeader_2.54mm:PinHeader_2x06_P2.54mm_Vertical; now fitted
Connections:
- net +3V3: now also J10.12 (Pin_12)
- net Bps_Hazard: now also J10.10 (Pin_10); no longer J10.9 (Pin_9)
- net Forward: now also J10.8 (Pin_8); no longer J10.7 (Pin_7)
- net GND: now also J10.1 (Pin_1)
- net Heartbeat: now also J10.11 (Pin_11); no longer J10.12 (Pin_12)
- net IG2: now also J10.7 (Pin_7); no longer J10.1 (Pin_1)
- net Reverse: now also J10.9 (Pin_9); no longer J10.8 (Pin_8)
- net UART4_Rx: no longer J10.11 (Pin_11)
- net UART4_Tx: no longer J10.10 (Pin_10)
Changed lines of the file:
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@@
 	(wire
 		(pts
+			(xy 118.11 175.26) (xy 118.11 177.8)
+		)
+		(stroke
+			(width 0)
+			(type default)
+		)
+	)
+	(wire
+		(pts
 			(xy 193.04 71.12) (xy 193.04 73.66)
 		)
@@
 	(wire
 		(pts
+			(xy 135.89 160.02) (xy 135.89 162.56)
+		)
+		(stroke
+			(width 0)
+			(type default)
+		)
+	)
+	(wire
+		(pts
 			(xy 218.44 113.03) (xy 215.9 113.03)
 		)
@@
 	)
 	(label "Heartbeat"
-		(at 135.89 162.56 0)
+		(at 135.89 165.1 0)
 		(fields_autoplaced yes)
 		(effects
@@
 		)
 	)
-	(label "UART4_Rx"
-		(at 135.89 165.1 0)
-		(fields_autoplaced yes)
-		(effects
-			(font
-				(size 1.27 1.27)
-			)
-			(justify left bottom)
-		)
-	)
 	(label "Right_Blink"
 		(at 74.93 201.93 0)
@@
 	)
 	(label "Forward"
-		(at 135.89 175.26 0)
+		(at 135.89 172.72 0)
 		(fields_autoplaced yes)
 		(effects
@@
 	)
 	(label "Reverse"
-		(at 135.89 172.72 0)
+		(at 135.89 170.18 0)
 		(fields_autoplaced yes)
 		(effects
@@
 	)
 	(label "Bps_Hazard"
-		(at 135.89 170.18 0)
+		(at 135.89 167.64 0)
 		(fields_autoplaced yes)
 		(effects
@@
 		)
 	)
-	(label "UART4_Tx"
-		(at 135.89 167.64 0)
-		(fields_autoplaced yes)
-		(effects
-			(font
-				(size 1.27 1.27)
-			)
-			(justify left bottom)
-		)
-	)
 	(label "PC13"
 		(at 283.21 200.66 180)
@@
 	)
 	(label "IG2"
-		(at 118.11 175.26 180)
+		(at 135.89 175.26 0)
 		(fields_autoplaced yes)
 		(effects
@@
 				(size 1.27 1.27)
 			)
-			(justify right bottom)
+			(justify left bottom)
 		)
 	)
@@
 	)
 	(symbol
+		(lib_id "power:GND")
+		(at 118.11 177.8 0)
+		(unit 1)
+		(exclude_from_sim no)
+		(in_bom yes)
+		(on_board yes)
+		(dnp no)
+		(property "Reference" "#PWR040"
+			(at 118.11 184.15 0)
+			(effects
+				(font
+					(size 1.27 1.27)
+				)
+				(hide yes)
+			)
+		)
+		(property "Value" "GND"
+			(at 118.237 182.1942 0)
+			(effects
+				(font
+					(size 1.27 1.27)
+				)
+			)
+		)
+		(property "Footprint" ""
+			(at 118.11 177.8 0)
+			(effects
+				(font
+					(size 1.27 1.27)
+				)
+				(hide yes)
+			)
+		)
+		(property "Datasheet" ""
+			(at 118.11 177.8 0)
+			(effects
+				(font
+					(size 1.27 1.27)
+				)
+				(hide yes)
+			)
+		)
+		(property "Description" "Power symbol creates a global label with name \"GND\" , ground"
+			(at 118.11 177.8 0)
+			(effects
+				(font
+					(size 1.27 1.27)
+				)
+				(hide yes)
+			)
+		)
+		(pin "1"
+		)
+		(instances
+			(project "Controls-Leader"
+				(path "/66218487-e316-4467-9eba-79d4626ab24e"
+					(reference "#PWR040")
+					(unit 1)
+				)
+			)
+		)
+	)
+	(symbol
 		(lib_id "Connector_Generic:Conn_02x06_Top_Bottom")
 		(at 125.73 170.18 0)
@@
 		(exclude_from_sim no)
 		(in_bom yes)
-		(on_board no)
-		(dnp yes)
+		(on_board yes)
+		(dnp no)
 		(property "Reference" "J10"
 			(at 127 181.61 0)
@@
 			)
 		)
-		(property "Footprint" "UTSVT_Connectors:Molex_MicroFit3.0_2x6xP3.00mm_PolarizingPeg_Vertical"
+		(property "Footprint" "Connector_PinHeader_2.54mm:PinHeader_2x06_P2.54mm_Vertical"
 			(at 125.73 170.18 0)
 			(effects
@@
 			)
 		)
-		(property "Footprint" "UTSVT_Connectors:Molex_MicroFit3.0_1x3xP3.00mm_PolarizingPeg_Vertical"
+		(property "Footprint" "Connector_PinHeader_2.54mm:PinHeader_1x03_P2.54mm_Vertical"
 			(at 345.44 173.99 0)
 			(effects
@@
 					(unit 1)
 				)
+			)
+		)
+	)
+	(symbol
+		(lib_id "power:+3.3V")
+		(at 135.89 160.02 0)
+		(unit 1)
+		(exclude_from_sim no)
+		(in_bom yes)
+		(on_board yes)
+		(dnp no)
+		(fields_autoplaced yes)
+		(property "Reference" "#PWR093"
+			(at 135.89 163.83 0)
+			(effects
+				(font
+					(size 1.27 1.27)
+				)
+				(hide yes)
+			)
+		)
+		(property "Value" "+3V3"
+			(at 135.89 154.94 0)
+			(effects
+				(font
+					(size 1.27 1.27)
+				)
+			)
+		)
+		(property "Footprint" ""
+			(at 135.89 160.02 0)
+			(effects
+				(font
+					(size 1.27 1.27)
+				)
+				(hide yes)
+			)
+		)
+		(property "Datasheet" ""
+			(at 135.89 160.02 0)
+			(effects
+				(font
+					(size 1.27 1.27)
+				)
+				(hide yes)
+			)
+		)
+		(property "Description" "Power symbol creates a global label with name \"+3.3V\""
+			(at 135.89 160.02 0)
+			(effects
+				(font
+					(size 1.27 1.27)
+				)
+				(hide yes)
+			)
+		)
+		(pin "1"
+		)
+		(instances
+			(project "Controls-Leader"
+				(path "/66218487-e316-4467-9eba-79d4626ab24e"
+					(reference "#PWR093")
+					(unit 1)
+				)
